Commit message: add codes packge

File: src/aubo_robot-Noetic/aubo_gazebo/urdf/aubo_pusher.xacro (robot description, xacro)
@@ -19,5 +19,5 @@
         <geometry>
             <!-- <cylinder length="0.18" radius="0.01"/> -->
-            <box size="0.04 0.04 0.18"/>
+            <box size="0.03 0.03 0.18"/>
         </geometry>
       </visual>
@@ -25,5 +25,5 @@
       <origin xyz="0 0 0" rpy="0 0 0" />
         <geometry>
-            <box size="0.04 0.04 0.18"/>
+            <box size="0.03 0.03 0.18"/>
         </geometry>
     </collision>
